Commit message: fix urdf

File: rm_simulation/pb_rm_simulation/urdf/simulation_waking_robot.xacro (robot description, xacro)
@@ -8,8 +8,8 @@
             <mass value="${mass}" />
             <inertia ixx="0.01" ixy="0.0" ixz="0.0"
-                    iyy="0.01" iyz="0.0" izz="0.01" />
+                     iyy="0.01" iyz="0.0" izz="0.01" />
         </inertial>
     </xacro:macro>
-    <link name="base_link">
+    <link name="chassis">
         <visual>
             <geometry>
@@ -29,9 +29,4 @@
         <xacro:default_inertial mass="8.2"/>
     </link>
-    <link name="base_link_fake" />
-    <joint name="base_link_to_base_link_fake" type="fixed">
-        <parent link="base_link" />
-        <child link="base_link_fake" />
-    </joint>
     <link name="wheel_1">
         <visual>
@@ -105,5 +100,5 @@
     </link>
     <joint name="base_to_wheel1" type="continuous">
-        <parent link="base_link"/>
+        <parent link="chassis"/>
         <child link="wheel_1"/>
         <origin rpy="${-PI/2} 0 0" xyz="0.1 0.13 0"/>
@@ -114,10 +109,10 @@
         <anchor xyz="0 0 0" />
         <limit effort="100" velocity="100" />
-        <parent link="base_link"/>
+        <parent link="chassis"/>
         <child link="wheel_2"/>
         <origin rpy="${-PI/2} 0 0" xyz="-0.1 0.13 0"/>
     </joint>
     <joint name="base_to_wheel3" type="continuous">
-        <parent link="base_link"/>
+        <parent link="chassis"/>
         <axis xyz="0 0 1" />
         <child link="wheel_3"/>
@@ -125,5 +120,5 @@
     </joint>
     <joint name="base_to_wheel4" type="continuous">
-        <parent link="base_link"/>
+        <parent link="chassis"/>
         <axis xyz="0 0 1" />
         <child link="wheel_4"/>
@@ -134,5 +129,5 @@
         <axis xyz="0 1 0" />
         <origin xyz="0.12 0 0.125" rpy="0 0 0"/>
-        <parent link="base_link"/>
+        <parent link="chassis"/>
         <child link="imu_link"/>
     </joint>
@@ -161,5 +156,5 @@
     </link>
     <!-- gazebo插件设置相关 -->
-    <gazebo reference="base_link">
+    <gazebo reference="chassis">
         <material>Gazebo/Orange</material>
     </gazebo>
@@ -226,5 +221,5 @@
     <!-- Livox-Mid360  -->
     <xacro:include filename="$(find ros2_livox_simulation)/urdf/mid360.xacro" />
-    <xacro:mid360 name="livox_frame" parent="base_link" topic="/livox/lidar">
+    <xacro:mid360 name="livox_frame" parent="chassis" topic="/livox/lidar">
         <origin xyz="0.12 0.0 0.175" rpy="0 0 0"/>
     </xacro:mid360>
